Commit message: refactor before adding new 🌍s

File: urdf/jenga_wall.urdf.xacro (robot description, xacro)
@@ -1,3 +1,3 @@
-<robot name="robot">
+<robot name="jenga_wall">
   <link name="jenga_wall_link">
     <inertial>
@@ -9,5 +9,5 @@
       <origin xyz="0 0 0" rpy="0 0 0" />
       <geometry>
-        <mesh filename="package://remaro_worlds/models/obstacles/jenga_wall.dae" />
+        <mesh filename="package://remaro_worlds/models/obstacles/jenga_wall/model.dae" />
       </geometry>
     </visual>
@@ -15,5 +15,5 @@
       <origin xyz="0 0 0" rpy="0 0 0" />
       <geometry>
-        <mesh filename="package://remaro_worlds/models/obstacles/jenga_wall.dae" />
+        <mesh filename="package://remaro_worlds/models/obstacles/jenga_wall/model.dae" />
       </geometry>
     </collision>
